Commit message: rotated xtion 360 degrees
The WPI-RAIL version of the youbot description had the xtion camera
facing in the opposite direction from the gripper. That's not how we
intend to use it, so here are updated xacro, urdf, and moveit config
files.

File: youbot_description/robots/youbot.urdf (robot description, URDF)
Before this commit: robot youbot, 29 links, 28 joints
Joints:
- joint gripper_palm_link_xtion_joint: origin xyz=0.0197188 -0.0341838 0.0459352 rpy=0.0201114 0.00763208 3.0937 -> xyz=-0.0100 0.0301838 0.0559352 rpy=0.0201114 0.00763208 -0.01789265

File: youbot_description/urdf/youbot_gripper/gripper.urdf.xacro (robot description, xacro)
@@ -126,5 +126,5 @@
 		<xacro:asus_xtion_camera name="xtion" parent="${name}_palm_link" tilt="0.0">
                   <!-- AR_CALIBRATOR:EDIT_HERE -->
-                  <origin xyz="0.0197188 -0.0341838 0.0459352" rpy="0.0201114 0.00763208 3.0937" />
+                  <origin xyz="-0.0100 0.0301838 0.0559352" rpy="0.0201114 0.00763208 -0.01789265" />
                 </xacro:asus_xtion_camera>
 		<!-- extensions -->
